File: PCB/ElephantV2.kicad_sch (KiCad schematic)
At the start: 45 parts, among them U1 Nice_Nano_V2

Commit message: commit
Parts:
- S00, S01, S02, S10, S11, S12, S20, S21, S22, S23, S30, S31, S32, S33, S40, S41, S42, S43, S50, S51, S52, S53: footprint ScottoKeebs_Hotswap:Hotswap_MX_1.00u_reversable -> Reversable_Rok_Prezelj:Choc_1.00u_reversable
Changed lines of the file:
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@@
 			)
 		)
-		(property "Footprint" "ScottoKeebs_Hotswap:Hotswap_MX_1.00u_reversable"
+		(property "Footprint" "Reversable_Rok_Prezelj:Choc_1.00u_reversable"
 			(at 133.985 95.25 0)
 			(effects
@@
 			)
 		)
-		(property "Footprint" "ScottoKeebs_Hotswap:Hotswap_MX_1.00u_reversable"
+		(property "Footprint" "Reversable_Rok_Prezelj:Choc_1.00u_reversable"
 			(at 149.225 74.295 0)
 			(effects
@@
 			)
 		)
-		(property "Footprint" "ScottoKeebs_Hotswap:Hotswap_MX_1.00u_reversable"
+		(property "Footprint" "Reversable_Rok_Prezelj:Choc_1.00u_reversable"
 			(at 118.745 37.465 0)
 			(effects
@@
 			)
 		)
-		(property "Footprint" "ScottoKeebs_Hotswap:Hotswap_MX_1.00u_reversable"
+		(property "Footprint" "Reversable_Rok_Prezelj:Choc_1.00u_reversable"
 			(at 149.225 37.465 0)
 			(effects
@@
 			)
 		)
-		(property "Footprint" "ScottoKeebs_Hotswap:Hotswap_MX_1.00u_reversable"
+		(property "Footprint" "Reversable_Rok_Prezelj:Choc_1.00u_reversable"
 			(at 118.745 95.25 0)
 			(effects
@@
 			)
 		)
-		(property "Footprint" "ScottoKeebs_Hotswap:Hotswap_MX_1.00u_reversable"
+		(property "Footprint" "Reversable_Rok_Prezelj:Choc_1.00u_reversable"
 			(at 149.225 95.25 0)
 			(effects
@@
 			)
 		)
-		(property "Footprint" "ScottoKeebs_Hotswap:Hotswap_MX_1.00u_reversable"
+		(property "Footprint" "Reversable_Rok_Prezelj:Choc_1.00u_reversable"
 			(at 88.9 74.295 0)
 			(effects
@@
 			)
 		)
-		(property "Footprint" "ScottoKeebs_Hotswap:Hotswap_MX_1.00u_reversable"
+		(property "Footprint" "Reversable_Rok_Prezelj:Choc_1.00u_reversable"
 			(at 164.465 74.295 0)
 			(effects
@@
 			)
 		)
-		(property "Footprint" "ScottoKeebs_Hotswap:Hotswap_MX_1.00u_reversable"
+		(property "Footprint" "Reversable_Rok_Prezelj:Choc_1.00u_reversable"
 			(at 118.745 74.295 0)
 			(effects
@@
 			)
 		)
-		(property "Footprint" "ScottoKeebs_Hotswap:Hotswap_MX_1.00u_reversable"
+		(property "Footprint" "Reversable_Rok_Prezelj:Choc_1.00u_reversable"
 			(at 104.14 37.465 0)
 			(effects
@@
 			)
 		)
-		(property "Footprint" "ScottoKeebs_Hotswap:Hotswap_MX_1.00u_reversable"
+		(property "Footprint" "Reversable_Rok_Prezelj:Choc_1.00u_reversable"
 			(at 133.985 74.295 0)
 			(effects
@@
 			)
 		)
-		(property "Footprint" "ScottoKeebs_Hotswap:Hotswap_MX_1.00u_reversable"
+		(property "Footprint" "Reversable_Rok_Prezelj:Choc_1.00u_reversable"
 			(at 104.14 55.245 0)
 			(effects
@@
 			)
 		)
-		(property "Footprint" "ScottoKeebs_Hotswap:Hotswap_MX_1.00u_reversable"
+		(property "Footprint" "Reversable_Rok_Prezelj:Choc_1.00u_reversable"
 			(at 133.985 37.465 0)
 			(effects
@@
 			)
 		)
-		(property "Footprint" "ScottoKeebs_Hotswap:Hotswap_MX_1.00u_reversable"
+		(property "Footprint" "Reversable_Rok_Prezelj:Choc_1.00u_reversable"
 			(at 88.9 37.465 0)
 			(effects
@@
 			)
 		)
-		(property "Footprint" "ScottoKeebs_Hotswap:Hotswap_MX_1.00u_reversable"
+		(property "Footprint" "Reversable_Rok_Prezelj:Choc_1.00u_reversable"
 			(at 104.14 74.295 0)
 			(effects
@@
 			)
 		)
-		(property "Footprint" "ScottoKeebs_Hotswap:Hotswap_MX_1.00u_reversable"
+		(property "Footprint" "Reversable_Rok_Prezelj:Choc_1.00u_reversable"
 			(at 118.745 55.245 0)
 			(effects
@@
 			)
 		)
-		(property "Footprint" "ScottoKeebs_Hotswap:Hotswap_MX_1.00u_reversable"
+		(property "Footprint" "Reversable_Rok_Prezelj:Choc_1.00u_reversable"
 			(at 164.465 95.25 0)
 			(effects
@@
 			)
 		)
-		(property "Footprint" "ScottoKeebs_Hotswap:Hotswap_MX_1.00u_reversable"
+		(property "Footprint" "Reversable_Rok_Prezelj:Choc_1.00u_reversable"
 			(at 164.465 37.465 0)
 			(effects
@@
 			)
 		)
-		(property "Footprint" "ScottoKeebs_Hotswap:Hotswap_MX_1.00u_reversable"
+		(property "Footprint" "Reversable_Rok_Prezelj:Choc_1.00u_reversable"
 			(at 88.9 55.245 0)
 			(effects
@@
 			)
 		)
-		(property "Footprint" "ScottoKeebs_Hotswap:Hotswap_MX_1.00u_reversable"
+		(property "Footprint" "Reversable_Rok_Prezelj:Choc_1.00u_reversable"
 			(at 133.985 55.245 0)
 			(effects
@@
 			)
 		)
-		(property "Footprint" "ScottoKeebs_Hotswap:Hotswap_MX_1.00u_reversable"
+		(property "Footprint" "Reversable_Rok_Prezelj:Choc_1.00u_reversable"
 			(at 149.225 55.245 0)
 			(effects
@@
 			)
 		)
-		(property "Footprint" "ScottoKeebs_Hotswap:Hotswap_MX_1.00u_reversable"
+		(property "Footprint" "Reversable_Rok_Prezelj:Choc_1.00u_reversable"
 			(at 164.465 55.245 0)
 			(effects
